Commit message: v0.0.1

File: snakebot_ws/src/snakebot/urdf/snakebot.urdf (robot description, URDF)
Before this commit: robot snakebot, 12 links, 11 joints
Links:
- removed link link_five
Joints:
- removed joint link_five_joint
- removed joint rod_six_joint

Commit message: v0.0.1

File: snakebot_ws/src/snakebot/urdf/snakebot.urdf (robot description, URDF)
Before this commit: robot snakebot, 11 links, 9 joints
Links:
- added link link_five, mass 0.372498080839688; collision mesh filename=package://snakebot/meshes/link_five.STL; visual mesh filename=package://snakebot/meshes/link_five.STL
Joints:
- added joint link_five_joint: type fixed, parent rod_six, child link_five, origin xyz=0 0.01 0 rpy=-1.5708 0 0, axis 0 0 1
- added joint rod_six_joint: type revolute, parent link_four, child rod_six, origin xyz=0.2159 0 0 rpy=0 0 0, axis 0 1 0, limit lower=-3.14 upper=3.14 effort=1000 velocity=0.1
